Commit message: complet

File: plat4m_description/urdf/plat4m.xacro (robot description, xacro)
@@ -25,10 +25,10 @@
   </collision>
 </link>
-<joint name="joint_0_1" type="fixed">
+<joint name="joint_0_1_l2" type="fixed">
   <origin xyz="0.50 0.0 0.01935" rpy="0.0 0.0 0.0"/>
   <parent link="link0_p4m"/>
-  <child link="link1_atache"/>
-</joint>
-<link name="link1_atache">
+  <child link="link1_atache_l2"/>
+</joint>
+<link name="link1_atache_l2">
   <inertial>
     <origin xyz="0.0 0.0 0.0" rpy="0.0 0.0 0.0"/>
@@ -53,11 +53,11 @@
   </collision>
 </link>
-<joint name="joint_1_2" type="continuous">
+<joint name="joint_1_2_l2" type="continuous">
   <origin xyz="0.000 0.000 0.021" rpy="0.0 0.0 0.0"/>
-  <parent link="link1_atache"/>
-  <child link="link2_act"/>
+  <parent link="link1_atache_l2"/>
+  <child link="link2_act_l2"/>
   <axis xyz="0.0 1.0 0.0"/>
 </joint>
-<link name="link2_act">
+<link name="link2_act_l2">
   <inertial>
     <origin xyz="0.0 0.0 0.0" rpy="0.0 0.0 0.0"/>
@@ -82,12 +82,12 @@
   </collision>
 </link>
-<joint name="joint_2_3" type="prismatic">
+<joint name="joint_2_3_l2" type="prismatic">
   <origin xyz="0.03 0.0 0.0" rpy="0.0 0.0 0.0"/>
-  <parent link="link2_act"/>
-  <child link="link3_tige"/>
+  <parent link="link2_act_l2"/>
+  <child link="link3_tige_l2"/>
   <axis xyz="1.0 0.0 0.0"/>
   <limit lower="0.000" upper="0.070" effort="100.0" velocity="20.0"/>
 </joint>
-<link name="link3_tige">
+<link name="link3_tige_l2">
   <inertial>
     <origin xyz="0.0 0.0 0.0" rpy="0.0 0.0 0.0"/>
@@ -112,5 +112,5 @@
   </collision>
 </link>
-<link name="link4_bras">
+<link name="link4_bras_l2">
   <inertial>
     <origin xyz="0.0 0.0 0.0" rpy="0.0 0.0 0.0"/>
@@ -135,17 +135,17 @@
   </collision>
 </link>
-<joint name="joint_0_5" type="fixed">
+<joint name="joint_0_5_l2" type="fixed">
   <origin xyz="0.65 0.0 0.01935" rpy="0.0 0.0 0.0"/>
   <parent link="link0_p4m"/>
-  <child link="link5_atpiv"/>
-</joint>
-<joint name="joint_4_5" type="revolute">
+  <child link="link5_atpiv_l2"/>
+</joint>
+<joint name="joint_4_5_l2" type="revolute">
   <origin xyz="0.0 0.0 0.0161" rpy="0.0 0.0 0.0"/>
-  <parent link="link5_atpiv"/>
-  <child link="link4_bras"/>
+  <parent link="link5_atpiv_l2"/>
+  <child link="link4_bras_l2"/>
   <axis xyz="0.0 1.0 0.0"/>
   <limit lower="0.000" upper="1" effort="100.0" velocity="20.0"/>
 </joint>
-<link name="link5_atpiv">
+<link name="link5_atpiv_l2">
   <inertial>
     <origin xyz="0.0 0.0 0.0" rpy="0.0 0.0 0.0"/>
@@ -170,11 +170,11 @@
   </collision>
 </link>
-<joint name="joint_5_6" type="continuous">
+<joint name="joint_5_6_l2" type="continuous">
   <origin xyz="0.120 0.000 -0.033" rpy="0.0 -0.27 0.0"/>
-  <parent link="link4_bras"/>
-  <child link="link6_roubi"/>
+  <parent link="link4_bras_l2"/>
+  <child link="link6_roubi_l2"/>
   <axis xyz="0.0 1.0 0.0"/>
 </joint>
-<link name="link6_roubi">
+<link name="link6_roubi_l2">
   <inertial>
     <origin xyz="0.0 0.0 0.0" rpy="0.0 0.0 0.0"/>
@@ -199,12 +199,12 @@
   </collision>
 </link>
-<joint name="joint_0_7" type="prismatic">
+<joint name="joint_0_7_l2" type="prismatic">
   <origin xyz="0.7 0.1 0.01935" rpy="0.0 0.0 0.0"/>
   <parent link="link0_p4m"/>
-  <child link="link7_brasimp"/>
+  <child link="link7_brasimp_l2"/>
   <axis xyz="1.0 0.0 0.0"/>
   <limit lower="0.0" upper="1.0" effort="20.0" velocity="20.0"/>
 </joint>
-<link name="link7_brasimp">
+<link name="link7_brasimp_l2">
   <inertial>
     <origin xyz="0.0 0.0 0.0" rpy="0.0 0.0 0.0"/>
@@ -229,11 +229,11 @@
   </collision>
 </link>
-<joint name="joint_7_8" type="continuous">
+<joint name="joint_7_8_l2" type="continuous">
   <origin xyz="0.0708 0.0 0.05" rpy="0.0 0.0 0.0"/>
-  <parent link="link7_brasimp"/>
-  <child link="link8_band"/>
+  <parent link="link7_brasimp_l2"/>
+  <child link="link8_band_l2"/>
   <axis xyz="0.0 0.0 1.0"/>
 </joint>
-<link name="link8_band">
+<link name="link8_band_l2">
   <inertial>
     <origin xyz="0.0 0.0 0.0" rpy="0.0 0.0 0.0"/>
@@ -258,4 +258,5 @@
   </collision>
 </link>
+<!-- _______________________________________________________________________________________________ -->
 <link name="link4_bras_l1">
   <inertial>
@@ -346,5 +347,5 @@
 </link>
 <joint name="joint_0_7_l1" type="prismatic">
-  <origin xyz="0.7 1.0 0.01935" rpy="0.0 0.0 0.0"/>
+  <origin xyz="0.7 0.95 0.01935" rpy="0.0 0.0 0.0"/>
   <parent link="link0_p4m"/>
   <child link="link7_brasimp_l1"/>
@@ -382,4 +383,680 @@
 </joint>
 <link name="link8_band_l1">
+  <inertial>
+    <origin xyz="0.0 0.0 0.0" rpy="0.0 0.0 0.0"/>
+    <mass value="0.0"/>
+    <inertia ixx="0.0" ixy="0.0" ixz="0.0" iyy="0.0" iyz="0.0" izz="0.0"/>
+  </inertial>
+  <visual name="">
+    <origin xyz="0.0 0.0 0.0" rpy="0.0 0.0 0.0"/>
+      <geometry>
+      <mesh filename="package://plat4m_description/meshes/link8_band.stl" scale="0.01 0.01 0.01"/>
+    </geometry>
+    <material name="">
+      <color rgba="1.0 0.0 0.0 1.0"/>
+      <texture filename=""/>
+    </material>
+  </visual>
+  <collision>
+    <origin xyz="0.0 0.0 0.0" rpy="0.0 0.0 0.0"/>
+    <geometry>
+      <mesh filename="package://plat4m_description/meshes/link8_band.stl" scale="0.01 0.01 0.01"/>
+    </geometry>
+  </collision>
+</link>
+<!-- _______________________________________________________________________________________________ -->
+<link name="link4_bras_l3">
+  <inertial>
+    <origin xyz="0.0 0.0 0.0" rpy="0.0 0.0 0.0"/>
+    <mass value="0.0"/>
+    <inertia ixx="0.0" ixy="0.0" ixz="0.0" iyy="0.0" iyz="0.0" izz="0.0"/>
+  </inertial>
+  <visual name="">
+    <origin xyz="0.0 0.0 0.0" rpy="0.0 0.0 0.0"/>
+      <geometry>
+      <mesh filename="package://plat4m_description/meshes/link4_bras.stl" scale="0.01 0.01 0.01"/>
+    </geometry>
+    <material name="">
+      <color rgba="1.0 0.0 0.0 1.0"/>
+      <texture filename=""/>
+    </material>
+  </visual>
+  <collision>
+    <origin xyz="0.0 0.0 0.0" rpy="0.0 0.0 0.0"/>
+    <geometry>
+      <mesh filename="package://plat4m_description/meshes/link4_bras.stl" scale="0.01 0.01 0.01"/>
+    </geometry>
+  </collision>
+</link>
+<joint name="joint_0_5_l3" type="fixed">
+  <origin xyz="0.65 -0.95 0.01935" rpy="0.0 0.0 0.0"/>
+  <parent link="link0_p4m"/>
+  <child link="link5_atpiv_l3"/>
+</joint>
+<joint name="joint_4_5_l3" type="revolute">
+  <origin xyz="0.0 0 0.0161" rpy="0.0 0.0 0.0"/>
+  <parent link="link5_atpiv_l3"/>
+  <child link="link4_bras_l3"/>
+  <axis xyz="0.0 1.0 0.0"/>
+  <limit lower="0.000" upper="1" effort="100.0" velocity="20.0"/>
+</joint>
+<link name="link5_atpiv_l3">
+  <inertial>
+    <origin xyz="0.0 0.0 0.0" rpy="0.0 0.0 0.0"/>
+    <mass value="0.0"/>
+    <inertia ixx="0.0" ixy="0.0" ixz="0.0" iyy="0.0" iyz="0.0" izz="0.0"/>
+  </inertial>
+  <visual name="">
+    <origin xyz="0.0 0.0 0.0" rpy="0.0 0.0 0.0"/>
+      <geometry>
+      <mesh filename="package://plat4m_description/meshes/link5_atpiv.stl" scale="0.01 0.01 0.01"/>
+    </geometry>
+    <material name="">
+      <color rgba="1.0 0.0 0.0 1.0"/>
+      <texture filename=""/>
+    </material>
+  </visual>
+  <collision>
+    <origin xyz="0.0 0.0 0.0" rpy="0.0 0.0 0.0"/>
+    <geometry>
+      <mesh filename="package://plat4m_description/meshes/link5_atpiv.stl" scale="0.01 0.01 0.01"/>
+    </geometry>
+  </collision>
+</link>
+<joint name="joint_5_6_l3" type="continuous">
+  <origin xyz="0.120 0 -0.033" rpy="0.0 -0.27 0.0"/>
+  <parent link="link4_bras_l3"/>
+  <child link="link6_roubi_l3"/>
+  <axis xyz="0.0 1.0 0.0"/>
+</joint>
+<link name="link6_roubi_l3">
+  <inertial>
+    <origin xyz="0.0 0.0 0.0" rpy="0.0 0.0 0.0"/>
+    <mass value="0.0"/>
+    <inertia ixx="0.0" ixy="0.0" ixz="0.0" iyy="0.0" iyz="0.0" izz="0.0"/>
+  </inertial>
+  <visual name="">
+    <origin xyz="0.0 0.0 0.0" rpy="0.0 0.0 0.0"/>
+      <geometry>
+      <mesh filename="package://plat4m_description/meshes/link6_roubi.stl" scale="0.01 0.01 0.01"/>
+    </geometry>
+    <material name="">
+      <color rgba="1.0 0.0 0.0 1.0"/>
+      <texture filename=""/>
+    </material>
+  </visual>
+  <collision>
+    <origin xyz="0.0 0.0 0.0" rpy="0.0 0.0 0.0"/>
+    <geometry>
+      <mesh filename="package://plat4m_description/meshes/link6_roubi.stl" scale="0.01 0.01 0.01"/>
+    </geometry>
+  </collision>
+</link>
+<joint name="joint_0_7_l3" type="prismatic">
+  <origin xyz="0.7 -0.9 0.01935" rpy="0.0 0.0 0.0"/>
+  <parent link="link0_p4m"/>
+  <child link="link7_brasimp_l3"/>
+  <axis xyz="1.0 0.0 0.0"/>
+  <limit lower="0.0" upper="1.0" effort="20.0" velocity="20.0"/>
+</joint>
+<link name="link7_brasimp_l3">
+  <inertial>
+    <origin xyz="0.0 0.0 0.0" rpy="0.0 0.0 0.0"/>
+    <mass value="0.0"/>
+    <inertia ixx="0.0" ixy="0.0" ixz="0.0" iyy="0.0" iyz="0.0" izz="0.0"/>
+  </inertial>
+  <visual name="">
+    <origin xyz="0.0 0.0 0.0" rpy="0.0 0.0 0.0"/>
+      <geometry>
+      <mesh filename="package://plat4m_description/meshes/link7_brasimp.stl" scale="0.01 0.01 0.01"/>
+    </geometry>
+    <material name="">
+      <color rgba="1.0 0.0 0.0 1.0"/>
+      <texture filename=""/>
+    </material>
+  </visual>
+  <collision>
+    <origin xyz="0.0 0.0 0.0" rpy="0.0 0.0 0.0"/>
+    <geometry>
+      <mesh filename="package://plat4m_description/meshes/link7_brasimp.stl" scale="0.01 0.01 0.01"/>
+    </geometry>
+  </collision>
+</link>
+<joint name="joint_7_8_l3" type="continuous">
+  <origin xyz="0.0708 0 0.05" rpy="0.0 0.0 0.0"/>
+  <parent link="link7_brasimp_l3"/>
+  <child link="link8_band_l3"/>
+  <axis xyz="0.0 0.0 1.0"/>
+</joint>
+<link name="link8_band_l3">
+  <inertial>
+    <origin xyz="0.0 0.0 0.0" rpy="0.0 0.0 0.0"/>
+    <mass value="0.0"/>
+    <inertia ixx="0.0" ixy="0.0" ixz="0.0" iyy="0.0" iyz="0.0" izz="0.0"/>
+  </inertial>
+  <visual name="">
+    <origin xyz="0.0 0.0 0.0" rpy="0.0 0.0 0.0"/>
+      <geometry>
+      <mesh filename="package://plat4m_description/meshes/link8_band.stl" scale="0.01 0.01 0.01"/>
+    </geometry>
+    <material name="">
+      <color rgba="1.0 0.0 0.0 1.0"/>
+      <texture filename=""/>
+    </material>
+  </visual>
+  <collision>
+    <origin xyz="0.0 0.0 0.0" rpy="0.0 0.0 0.0"/>
+    <geometry>
+      <mesh filename="package://plat4m_description/meshes/link8_band.stl" scale="0.01 0.01 0.01"/>
+    </geometry>
+  </collision>
+</link>
+<!---->
+<!---->
+<joint name="joint_0_1_r2" type="fixed">
+  <origin xyz="-0.50 0.0 0.01935" rpy="0.0 0.0 3.1416"/>
+  <parent link="link0_p4m"/>
+  <child link="link1_atache_r2"/>
+</joint>
+<link name="link1_atache_r2">
+  <inertial>
+    <origin xyz="0.0 0.0 0.0" rpy="0.0 0.0 0.0"/>
+    <mass value="0.0"/>
+    <inertia ixx="0.0" ixy="0.0" ixz="0.0" iyy="0.0" iyz="0.0" izz="0.0"/>
+  </inertial>
+  <visual name="">
+    <origin xyz="0.0 0.0 0.0" rpy="0.0 0.0 0.0"/>
+    <geometry>
+      <mesh filename="package://plat4m_description/meshes/link1_atache.stl" scale="0.01 0.01 0.01"/>
+    </geometry>
+    <material name="">
+      <color rgba="1.0 0.0 0.0 1.0"/>
+      <texture filename=""/>
+    </material>
+  </visual>
+  <collision>
+    <origin xyz="0.0 0.0 0.0" rpy="0.0 0.0 0.0"/>
+    <geometry>
+      <mesh filename="package://plat4m_description/meshes/link1_atache.stl" scale="0.01 0.01 0.01"/>
+    </geometry>
+  </collision>
+</link>
+<joint name="joint_1_2_r2" type="continuous">
+  <origin xyz="0.000 0.000 0.021" rpy="0.0 0.0 0.0"/>
+  <parent link="link1_atache_r2"/>
+  <child link="link2_act_r2"/>
+  <axis xyz="0.0 1.0 0.0"/>
+</joint>
+<link name="link2_act_r2">
+  <inertial>
+    <origin xyz="0.0 0.0 0.0" rpy="0.0 0.0 0.0"/>
+    <mass value="0.0"/>
+    <inertia ixx="0.0" ixy="0.0" ixz="0.0" iyy="0.0" iyz="0.0" izz="0.0"/>
+  </inertial>
+  <visual name="">
+    <origin xyz="0.0 0.0 0.0" rpy="0.0 0.0 0.0"/>
+    <geometry>
+      <mesh filename="package://plat4m_description/meshes/link2_act.stl" scale="0.01 0.01 0.01"/>
+       </geometry>
+    <material name="">
+      <color rgba="1.0 0.0 0.0 1.0"/>
+      <texture filename=""/>
+    </material>
+  </visual>
+  <collision>
+    <origin xyz="0.0 0.0 0.0" rpy="0.0 0.0 0.0"/>
+    <geometry>
+      <mesh filename="package://plat4m_description/meshes/link2_act.stl" scale="0.01 0.01 0.01"/>
+    </geometry>
+  </collision>
+</link>
+<joint name="joint_2_3_r2" type="prismatic">
+  <origin xyz="0.03 0.0 0.0" rpy="0.0 0.0 0.0"/>
+  <parent link="link2_act_r2"/>
+  <child link="link3_tige_r2"/>
+  <axis xyz="1.0 0.0 0.0"/>
+  <limit lower="0.000" upper="0.070" effort="100.0" velocity="20.0"/>
+</joint>
+<link name="link3_tige_r2">
+  <inertial>
+    <origin xyz="0.0 0.0 0.0" rpy="0.0 0.0 0.0"/>
+    <mass value="0.0"/>
+    <inertia ixx="0.0" ixy="0.0" ixz="0.0" iyy="0.0" iyz="0.0" izz="0.0"/>
+  </inertial>
+  <visual name="">
+    <origin xyz="0.0 0.0 0.0" rpy="0.0 0.0 0.0"/>
+      <geometry>
+      <mesh filename="package://plat4m_description/meshes/link3_tige.stl" scale="0.01 0.01 0.01"/>
+    </geometry>
+    <material name="">
+      <color rgba="1.0 0.0 0.0 1.0"/>
+      <texture filename=""/>
+    </material>
+  </visual>
+  <collision>
+    <origin xyz="0.0 0.0 0.0" rpy="0.0 0.0 0.0"/>
+    <geometry>
+      <mesh filename="package://plat4m_description/meshes/link3_tige.stl" scale="0.01 0.01 0.01"/>
+    </geometry>
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
Commit message: joint a point

File: plat4m_description/urdf/plat4m.xacro (robot description, xacro)
@@ -144,5 +144,5 @@
   <parent link="link5_atpiv_l2"/>
   <child link="link4_bras_l2"/>
-  <axis xyz="0.0 1.0 0.0"/>
+  <axis xyz="0.0 -1.0 0.0"/>
   <limit lower="0.000" upper="1" effort="100.0" velocity="20.0"/>
 </joint>
@@ -174,5 +174,5 @@
   <parent link="link4_bras_l2"/>
   <child link="link6_roubi_l2"/>
-  <axis xyz="0.0 1.0 0.0"/>
+  <axis xyz="1.0 0.0 0.0"/>
 </joint>
 <link name="link6_roubi_l2">
@@ -203,6 +203,6 @@
   <parent link="link0_p4m"/>
   <child link="link7_brasimp_l2"/>
-  <axis xyz="1.0 0.0 0.0"/>
-  <limit lower="0.0" upper="1.0" effort="20.0" velocity="20.0"/>
+  <axis xyz="-1.0 0.0 0.0"/>
+  <limit lower="0.0" upper="0.1" effort="20.0" velocity="20.0"/>
 </joint>
 <link name="link7_brasimp_l2">
@@ -291,5 +291,5 @@
   <parent link="link5_atpiv_l1"/>
   <child link="link4_bras_l1"/>
-  <axis xyz="0.0 1.0 0.0"/>
+  <axis xyz="0.0 -1.0 0.0"/>
   <limit lower="0.000" upper="1" effort="100.0" velocity="20.0"/>
 </joint>
@@ -321,5 +321,5 @@
   <parent link="link4_bras_l1"/>
   <child link="link6_roubi_l1"/>
-  <axis xyz="0.0 1.0 0.0"/>
+  <axis xyz="1.0 0.0 0.0"/>
 </joint>
 <link name="link6_roubi_l1">
@@ -350,6 +350,6 @@
   <parent link="link0_p4m"/>
   <child link="link7_brasimp_l1"/>
-  <axis xyz="1.0 0.0 0.0"/>
-  <limit lower="0.0" upper="1.0" effort="20.0" velocity="20.0"/>
+  <axis xyz="-1.0 0.0 0.0"/>
+  <limit lower="0.0" upper="0.1" effort="20.0" velocity="20.0"/>
 </joint>
 <link name="link7_brasimp_l1">
@@ -438,5 +438,5 @@
   <parent link="link5_atpiv_l3"/>
   <child link="link4_bras_l3"/>
-  <axis xyz="0.0 1.0 0.0"/>
+  <axis xyz="0.0 -1.0 0.0"/>
   <limit lower="0.000" upper="1" effort="100.0" velocity="20.0"/>
 </joint>
@@ -468,5 +468,5 @@
   <parent link="link4_bras_l3"/>
   <child link="link6_roubi_l3"/>
-  <axis xyz="0.0 1.0 0.0"/>
+  <axis xyz="1.0 0.0 0.0"/>
 </joint>
 <link name="link6_roubi_l3">
@@ -497,6 +497,6 @@
   <parent link="link0_p4m"/>
   <child link="link7_brasimp_l3"/>
-  <axis xyz="1.0 0.0 0.0"/>
-  <limit lower="0.0" upper="1.0" effort="20.0" velocity="20.0"/>
+  <axis xyz="-1.0 0.0 0.0"/>
+  <limit lower="0.0" upper="0.1" effort="20.0" velocity="20.0"/>
 </joint>
 <link name="link7_brasimp_l3">
@@ -673,5 +673,5 @@
   <parent link="link5_atpiv_r2"/>
   <child link="link4_bras_r2"/>
-  <axis xyz="0.0 1.0 0.0"/>
+  <axis xyz="0.0 -1.0 0.0"/>
   <limit lower="0.000" upper="1" effort="100.0" velocity="20.0"/>
 </joint>
@@ -703,5 +703,5 @@
   <parent link="link4_bras_r2"/>
   <child link="link6_roubi_r2"/>
-  <axis xyz="0.0 1.0 0.0"/>
+  <axis xyz="-1.0 0.0 0.0"/>
 </joint>
 <link name="link6_roubi_r2">
@@ -732,6 +732,6 @@
   <parent link="link0_p4m"/>
   <child link="link7_brasimp_r2"/>
-  <axis xyz="1.0 0.0 0.0"/>
-  <limit lower="0.0" upper="1.0" effort="20.0" velocity="20.0"/>
+  <axis xyz="-1.0 0.0 0.0"/>
+  <limit lower="0.0" upper="0.1" effort="20.0" velocity="20.0"/>
 </joint>
 <link name="link7_brasimp_r2">
@@ -820,5 +820,5 @@
   <parent link="link5_atpiv_r1"/>
   <child link="link4_bras_r1"/>
-  <axis xyz="0.0 1.0 0.0"/>
+  <axis xyz="0.0 -1.0 0.0"/>
   <limit lower="0.000" upper="1" effort="100.0" velocity="20.0"/>
 </joint>
@@ -850,5 +850,5 @@
   <parent link="link4_bras_r1"/>
   <child link="link6_roubi_r1"/>
-  <axis xyz="0.0 1.0 0.0"/>
+  <axis xyz="1.0 0.0 0.0"/>
 </joint>
 <link name="link6_roubi_r1">
@@ -876,9 +876,9 @@
 </link>
 <joint name="joint_0_7_r1" type="prismatic">
-  <origin xyz="-0.7 0.95 0.01935" rpy="0.0 0.0 0.0"/>
+  <origin xyz="-0.7 0.95 0.01935" rpy="0.0 0.0 3.1416"/>
   <parent link="link0_p4m"/>
   <child link="link7_brasimp_r1"/>
-  <axis xyz="1.0 0.0 0.0"/>
-  <limit lower="0.0" upper="1.0" effort="20.0" velocity="20.0"/>
+  <axis xyz="-1.0 0.0 0.0"/>
+  <limit lower="0.0" upper="0.1" effort="20.0" velocity="20.0"/>
 </joint>
 <link name="link7_brasimp_r1">
@@ -967,5 +967,5 @@
   <parent link="link5_atpiv_r3"/>
   <child link="link4_bras_r3"/>
-  <axis xyz="0.0 1.0 0.0"/>
+  <axis xyz="0.0 -1.0 0.0"/>
   <limit lower="0.000" upper="1" effort="100.0" velocity="20.0"/>
 </joint>
@@ -997,5 +997,5 @@
   <parent link="link4_bras_r3"/>
   <child link="link6_roubi_r3"/>
-  <axis xyz="0.0 1.0 0.0"/>
+  <axis xyz="1.0 0.0 0.0"/>
 </joint>
 <link name="link6_roubi_r3">
@@ -1026,6 +1026,6 @@
   <parent link="link0_p4m"/>
   <child link="link7_brasimp_r3"/>
-  <axis xyz="1.0 0.0 0.0"/>
-  <limit lower="0.0" upper="1.0" effort="20.0" velocity="20.0"/>
+  <axis xyz="-1.0 0.0 0.0"/>
+  <limit lower="0.0" upper="0.1" effort="20.0" velocity="20.0"/>
 </joint>
 <link name="link7_brasimp_r3">

Commit message: position joint

File: plat4m_description/urdf/plat4m.xacro (robot description, xacro)
@@ -347,5 +347,5 @@
 </link>
 <joint name="joint_0_7_l1" type="prismatic">
-  <origin xyz="0.7 0.95 0.01935" rpy="0.0 0.0 0.0"/>
+  <origin xyz="0.7 0.98 0.01935" rpy="0.0 0.0 0.0"/>
   <parent link="link0_p4m"/>
   <child link="link7_brasimp_l1"/>
@@ -430,5 +430,5 @@
 </link>
 <joint name="joint_0_5_l3" type="fixed">
-  <origin xyz="0.65 -0.95 0.01935" rpy="0.0 0.0 0.0"/>
+  <origin xyz="0.65 -0.9 0.01935" rpy="0.0 0.0 0.0"/>
   <parent link="link0_p4m"/>
   <child link="link5_atpiv_l3"/>
@@ -494,5 +494,5 @@
 </link>
 <joint name="joint_0_7_l3" type="prismatic">
-  <origin xyz="0.7 -0.9 0.01935" rpy="0.0 0.0 0.0"/>
+  <origin xyz="0.7 -0.98 0.01935" rpy="0.0 0.0 0.0"/>
   <parent link="link0_p4m"/>
   <child link="link7_brasimp_l3"/>
@@ -876,5 +876,5 @@
 </link>
 <joint name="joint_0_7_r1" type="prismatic">
-  <origin xyz="-0.7 0.95 0.01935" rpy="0.0 0.0 3.1416"/>
+  <origin xyz="-0.7 0.98 0.01935" rpy="0.0 0.0 3.1416"/>
   <parent link="link0_p4m"/>
   <child link="link7_brasimp_r1"/>
@@ -959,5 +959,5 @@
 </link>
 <joint name="joint_0_5_r3" type="fixed">
-  <origin xyz="-0.65 -0.95 0.01935" rpy="0.0 0.0 3.1416"/>
+  <origin xyz="-0.65 -0.9 0.01935" rpy="0.0 0.0 3.1416"/>
   <parent link="link0_p4m"/>
   <child link="link5_atpiv_r3"/>
@@ -1023,5 +1023,5 @@
 </link>
 <joint name="joint_0_7_r3" type="prismatic">
-  <origin xyz="-0.7 -0.9 0.01935" rpy="0.0 0.0 3.1416"/>
+  <origin xyz="-0.7 -0.98 0.01935" rpy="0.0 0.0 3.1416"/>
   <parent link="link0_p4m"/>
   <child link="link7_brasimp_r3"/>
